File: opennugget.kicad_sch (KiCad schematic)
At the start: 0 parts

Commit message: Updated files (need to organize)
Parts:
- added U4: RASPBERRY_PI_ZERO_2_W, RASPBERRY_PI_ZERO_2_W:MODULE_RASPBERRY_PI_ZERO_2_W, symbol RASPBERRY_PI_ZERO_2_W:RASPBERRY_PI_ZERO_2_W
Other:
- added sheet audio_out (temp.kicad_sch)
- added sheet clickwheel (clickwheel.kicad_sch)
- added sheet display (display.kicad_sch)
- added sheet power_IO (power_IO.kicad_sch)
